File: MiniPiano/MiniPiano.sch (KiCad schematic (older format))
At the start: 39 parts, among them J1 POWER, J2 SW_D5, J3 SW_F5, J4 SW_G5, J5 SW_A5, J6 SW_C6, J7 SW_D6, J8 OUT, U1 40106

Commit message: pictures
Other:
- note added: "Adjust for 739,98 Hz"
- note added: "F#5"
- note removed: "Adjust for 698,46 Hz"
- note removed: "F5"
Changed lines of the file:
@@
 D5
 Text Notes 3100 3800 0    50   ~ 0
-F5
+F#5
 Text Notes 4500 3800 0    50   ~ 0
 G5
@@
 Adjust for 587,33 Hz
 Text Notes 2550 2750 0    50   ~ 0
-Adjust for 698,46 Hz
+Adjust for 739,98 Hz
 Text Notes 4000 2750 0    50   ~ 0
 Adjust for 784 Hz

Commit message: fix valores de resistencias
Parts:
- R10: value 12k -> 18k
- R14: value 8.2k -> 10k
- R15: value 6.8k -> 8.2k
Changed lines of the file:
@@
 P 4100 3000
 F 0 "R10" V 3893 3000 50  0000 C CNN
-F 1 "12k" V 3984 3000 50  0000 C CNN
+F 1 "18k" V 3984 3000 50  0000 C CNN
 F 2 "Resistor_THT:R_Axial_DIN0204_L3.6mm_D1.6mm_P7.62mm_Horizontal" V 4030 3000 50  0001 C CNN
 F 3 "~" H 4100 3000 50  0001 C CNN
@@
 P 6950 3000
 F 0 "R14" V 6743 3000 50  0000 C CNN
-F 1 "8.2k" V 6834 3000 50  0000 C CNN
+F 1 "10k" V 6834 3000 50  0000 C CNN
 F 2 "Resistor_THT:R_Axial_DIN0204_L3.6mm_D1.6mm_P7.62mm_Horizontal" V 6880 3000 50  0001 C CNN
 F 3 "~" H 6950 3000 50  0001 C CNN
@@
 P 8400 3000
 F 0 "R15" V 8193 3000 50  0000 C CNN
-F 1 "6.8k" V 8284 3000 50  0000 C CNN
+F 1 "8.2k" V 8284 3000 50  0000 C CNN
 F 2 "Resistor_THT:R_Axial_DIN0204_L3.6mm_D1.6mm_P7.62mm_Horizontal" V 8330 3000 50  0001 C CNN
 F 3 "~" H 8400 3000 50  0001 C CNN

Commit message: fix resistencias
Parts:
- R11: value 3.3k -> 470
Changed lines of the file:
@@
 P 4450 7000
 F 0 "R11" H 4380 6954 50  0000 R CNN
-F 1 "3.3k" H 4380 7045 50  0000 R CNN
+F 1 "470" H 4380 7045 50  0000 R CNN
 F 2 "Resistor_THT:R_Axial_DIN0204_L3.6mm_D1.6mm_P7.62mm_Horizontal" V 4380 7000 50  0001 C CNN
 F 3 "~" H 4450 7000 50  0001 C CNN
